Commit message: gui implemented and working on server

File: webots/controllers/BlockArm/BlockArm.old.urdf (robot description, URDF)
Before this commit: robot D:/school/CPSC_Courses/CPSC_354/pulse/webots/controllers/BlockArm/Robot.urdf, 24 links, 23 joints
Links:
- removed link gps
- removed link inertial unit
- removed link solid_7
- link solid_6: geometry collision box size=0.05 0.05 0.05; visual box size=0.05 0.05 0.05
Joints:
- removed joint ROBOTIQ 2F-140 Gripper_inertial unit_joint
- removed joint base_link_gps_joint
- removed joint hingejoint_10
- removed joint solid_7_ROBOTIQ 2F-140 Gripper_joint
- removed joint wrist2_motor
- added joint hingejoint_7: type revolute, parent right outer finger, child ROBOTIQ 2F-140 Gripper right inner finger, origin xyz=0 0.081755 -0.0282 rpy=-0.725 0 0, axis 1 0 0
- added joint solid_6_ROBOTIQ 2F-140 Gripper_joint: type fixed, parent solid_6, child ROBOTIQ 2F-140 Gripper, origin xyz=0 0 0 rpy=0 0 0
- joint hingejoint_8: child ROBOTIQ 2F-140 Gripper right inner finger -> left inner knuckle; origin xyz=0 0.081755 -0.0282 rpy=-0.725 0 0 -> xyz=0 -0.0127 0.06142 rpy=2.295796 0 0; parent right outer finger -> ROBOTIQ 2F-140 Gripper
- joint hingejoint_9: child left inner knuckle -> ROBOTIQ 2F-140 Gripper left inner finger; origin xyz=0 -0.0127 0.06142 rpy=2.295796 0 0 -> xyz=0 0.081755 -0.02822 rpy=-0.725 0 0; parent ROBOTIQ 2F-140 Gripper -> left outer finger
- joint solid_5_solid_6_joint: origin xyz=-0.06 0 0 rpy=0 0 0 -> xyz=0 0 0.03 rpy=0 0 0
- joint wrist_motor: axis 1 0 0 -> 0 0 1
